File: schematic/mePed.sch (EAGLE design)
At the start: 34 parts, among them IC1 MEGA328-PU, Q1 16MHz, X1 Power

Commit message: Add files via upload
Parts:
- added S2: Reset, switch-omron:10-XX
Connections:
- net GND: now also S2.P, S2.P1
- net N$2: now also S2.S, S2.S1
Other:
- moved on the sheet: LED1
Changed lines of the file:
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@@
 <part name="SUPPLY9" library="supply2" deviceset="GND" device=""/>
 <part name="X1" library="con-ptr500" deviceset="AK300/2" device="" value="Power"/>
+<part name="S2" library="switch-omron" deviceset="10-XX" device="" value="Reset"/>
 </parts>
 <sheets>
@@
 <instance part="R6" gate="G$1" x="-22.86" y="99.06"/>
 <instance part="R7" gate="G$1" x="12.7" y="5.08" rot="R90"/>
-<instance part="LED1" gate="G$1" x="-33.02" y="93.98"/>
+<instance part="LED1" gate="G$1" x="-33.02" y="96.52"/>
 <instance part="LED2" gate="G$1" x="12.7" y="-2.54"/>
 <instance part="SUPPLY7" gate="GND" x="12.7" y="-10.16"/>
@@
 <instance part="X1" gate="-1" x="-38.1" y="-10.16"/>
 <instance part="X1" gate="-2" x="-38.1" y="-15.24"/>
+<instance part="S2" gate="1" x="-17.78" y="88.9" rot="R270"/>
 </instances>
 <busses>
@@
 <junction x="-33.02" y="33.02"/>
 <pinref part="LED1" gate="G$1" pin="C"/>
+<wire x1="-33.02" y1="91.44" x2="-33.02" y2="88.9" width="0.1524" layer="91"/>
+<junction x="-33.02" y="73.66"/>
+<pinref part="S2" gate="1" pin="P1"/>
+<pinref part="S2" gate="1" pin="P"/>
 <wire x1="-33.02" y1="88.9" x2="-33.02" y2="73.66" width="0.1524" layer="91"/>
-<junction x="-33.02" y="73.66"/>
+<wire x1="-22.86" y1="88.9" x2="-22.86" y2="86.36" width="0.1524" layer="91"/>
+<wire x1="-22.86" y1="88.9" x2="-33.02" y2="88.9" width="0.1524" layer="91"/>
+<junction x="-33.02" y="88.9"/>
+<junction x="-22.86" y="88.9"/>
 </segment>
 <segment>
@@
 <pinref part="JP2" gate="G$1" pin="5"/>
 <wire x1="-15.24" y1="20.32" x2="0" y2="20.32" width="0.1524" layer="91"/>
+<pinref part="S2" gate="1" pin="S"/>
+<wire x1="0" y1="88.9" x2="-12.7" y2="88.9" width="0.1524" layer="91"/>
+<pinref part="S2" gate="1" pin="S1"/>
+<wire x1="-12.7" y1="88.9" x2="-12.7" y2="86.36" width="0.1524" layer="91"/>
+<junction x="-12.7" y="88.9"/>
 </segment>
 </net>
@@
 <pinref part="LED1" gate="G$1" pin="A"/>
 <wire x1="-27.94" y1="99.06" x2="-33.02" y2="99.06" width="0.1524" layer="91"/>
-<wire x1="-33.02" y1="99.06" x2="-33.02" y2="96.52" width="0.1524" layer="91"/>
-</segment>
-</net>
+</segment>
+</net>
